File: pcb/desk_winder.brd (EAGLE design)
At the start: 161.3 x 100 mm, 14 parts, among them IC1 TINY13-20PU, IC2 7805L, J1 22-27-2041-04, X1 22-23-2021, X2 22-23-2031

Commit message: pcb
Parts:
- C1, C2: device rcl:C025-024X044 -> rcl:C050-025X075
- R2: value 4.7k -> 8.2k; device resistor:0207/10 -> resistor:0207/12
- R4, R7, R9: device resistor:0207/10 -> resistor:0207/12
- moved R9 8.98 mm to (40.6, 11.4), turned to 90 degrees
- moved R2 8.89 mm to (30.5, 14.0), turned to 270 degrees
- moved C1 6.84 mm to (19.1, 21.6)
- moved R7 6.48 mm to (35.6, 15.2), turned to 270 degrees
- moved R4 4.02 mm to (30.5, 5.08)
- moved C2 3.81 mm to (22.9, 14.0), turned to 0 degrees
- moved IC2 2.54 mm to (16.5, 16.5)
- moved D1 1.27 mm to (8.89, 21.6)
- moved IC1 1.27 mm to (14.0, 7.62)
Routing:
- net VCC: track 34.8 -> 41.6 mm
- net +12V: track 51.6 -> 46.0 mm
- net SENSE: track 15.8 -> 10.7 mm
- net TACH_IN: track 10.7 -> 15.0 mm
- net N$1: track 5.08 -> 8.89 mm
- net VDD: track 3.81 -> 5.08 mm
- net POTZ: track 7.62 -> 6.35 mm
- net CTRL: track 29.0 -> 30.3 mm
- net GND: track 0.00 -> 1.27 mm

Commit message: pcb
Parts:
- moved LED1 5.08 mm to (40.6, 21.6)
Routing:
- net N$1: track 8.89 -> 3.81 mm
- net VCC: track 41.6 -> 40.3 mm
- net GND: track 1.27 -> 0.00 mm
- net SENSE: track 10.7 -> 11.4 mm
- net CTRL: track 30.3 -> 31.0 mm
Other:
- board size 161.3 x 100 mm -> 53.3 x 25.1 mm

Commit message: WIP from AVR442
Parts:
- R2: value 8.2k -> 10k
Connections:
- net CTRL renamed PWM
Changed lines of the file:
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@@
 <layer number="19" name="Unrouted" color="6" fill="1" visible="no" active="yes"/>
 <layer number="20" name="Dimension" color="15" fill="1" visible="no" active="yes"/>
-<layer number="21" name="tPlace" color="7" fill="1" visible="no" active="yes"/>
+<layer number="21" name="tPlace" color="7" fill="1" visible="yes" active="yes"/>
 <layer number="22" name="bPlace" color="7" fill="1" visible="no" active="yes"/>
 <layer number="23" name="tOrigins" color="15" fill="1" visible="no" active="yes"/>
 <layer number="24" name="bOrigins" color="15" fill="1" visible="no" active="yes"/>
-<layer number="25" name="tNames" color="7" fill="1" visible="no" active="yes"/>
+<layer number="25" name="tNames" color="7" fill="1" visible="yes" active="yes"/>
 <layer number="26" name="bNames" color="7" fill="1" visible="no" active="yes"/>
-<layer number="27" name="tValues" color="7" fill="1" visible="no" active="yes"/>
+<layer number="27" name="tValues" color="7" fill="1" visible="yes" active="yes"/>
 <layer number="28" name="bValues" color="7" fill="1" visible="no" active="yes"/>
 <layer number="29" name="tStop" color="7" fill="3" visible="no" active="yes"/>
@@
 <attribute name="OC_FARNELL" value="9171550" x="13.97" y="7.62" size="1.778" layer="27" rot="R270" display="off"/>
 </element>
-<element name="R2" library="resistor" package="0207/12" value="8.2k" x="30.48" y="13.97" rot="R270"/>
+<element name="R2" library="resistor" package="0207/12" value="10k" x="30.48" y="13.97" rot="R270"/>
 <element name="R4" library="resistor" package="0207/12" value="10k" x="30.48" y="5.08"/>
 <element name="R7" library="resistor" package="0207/12" value="200" x="35.56" y="15.24" rot="R270"/>
@@
 <wire x1="39.37" y1="21.59" x2="35.56" y2="21.59" width="0.635" layer="16"/>
 </signal>
-<signal name="CTRL">
+<signal name="PWM">
 <contactref element="IC1" pad="5"/>
 <contactref element="J1" pad="4"/>
